Commit message: update turret

File: bras/urdf/turret.urdf (robot description, URDF)
Before this commit: robot turret, 6 links, 5 joints
Joints:
- joint joint2: origin xyz=0. 0 0.0 rpy=1.57079632679 0 0 -> xyz=0. 0 0.0 rpy=-1.57079632679 0 0

Commit message: update turret

File: bras/urdf/turret.urdf (robot description, URDF)
Before this commit: robot turret, 6 links, 5 joints
Joints:
- joint joint2: axis 0 0 1 -> 0 0 -1; origin xyz=0. 0 0.0 rpy=-1.57079632679 0 0 -> xyz=0. 0 0.0 rpy=1.57079632679 0 0
